Commit message: genetic algorithm added. next to convert to URDF for use with pybullet

File: test.urdf (robot description, URDF)
Before this commit: robot my_first, 2 links, 1 joints
Links:
- added link sub_link2, mass 0.25; collision cylinder length=5 radius=1.25; visual cylinder length=5 radius=0.1
- link base_link: geometry collision cylinder length=0.6 radius=0.25; visual cylinder length=0.6 radius=0.25
- link sub_link: geometry collision cylinder length=1 radius=1.25; visual cylinder length=1 radius=0.1
Joints:
- added joint base_to_sub2: type revolute, parent base_link, child sub_link2, origin xyz=0.5 0 0 rpy=0 0 0, axis 1 0 0, limit lower=0 upper=10 effort=10 velocity=1
- joint base_to_sub: axis (none) -> 1 0 0; limit (none) -> lower=0 upper=10 effort=10 velocity=1; origin (none) -> xyz=0.5 0 0 rpy=0 0 0; type fixed -> revolute

Commit message: pybullet simulation working from genetic algorithm

File: test.urdf (robot description, URDF)
Before this commit: robot myfirst, 3 links, 2 joints
Links:
- removed link base_link
- removed link sub_link
- removed link sub_link2
- added link 0, mass 0.16128612039875004; collision cylinder length=0.31219260664229476 radius=0.4055199778035763; visual cylinder length=0.31219260664229476 radius=0.4055199778035763
- added link 11, mass 0.04366996950557373; collision cylinder length=0.4726183526003428 radius=0.17149885188383895; visual cylinder length=0.4726183526003428 radius=0.17149885188383895
- added link 14, mass 0.04366996950557373; collision cylinder length=0.4726183526003428 radius=0.17149885188383895; visual cylinder length=0.4726183526003428 radius=0.17149885188383895
- added link 17, mass 0.04366996950557373; collision cylinder length=0.4726183526003428 radius=0.17149885188383895; visual cylinder length=0.4726183526003428 radius=0.17149885188383895
- added link 22, mass 0.24003132671428143; collision cylinder length=0.8673625771967088 radius=0.29679643923896615; visual cylinder length=0.8673625771967088 radius=0.29679643923896615
- added link 23, mass 0.24003132671428143; collision cylinder length=0.8673625771967088 radius=0.29679643923896615; visual cylinder length=0.8673625771967088 radius=0.29679643923896615
- added link 25, mass 0.24003132671428143; collision cylinder length=0.8673625771967088 radius=0.29679643923896615; visual cylinder length=0.8673625771967088 radius=0.29679643923896615
- added link 26, mass 0.24003132671428143; collision cylinder length=0.8673625771967088 radius=0.29679643923896615; visual cylinder length=0.8673625771967088 radius=0.29679643923896615
- added link 28, mass 0.24003132671428143; collision cylinder length=0.8673625771967088 radius=0.29679643923896615; visual cylinder length=0.8673625771967088 radius=0.29679643923896615
- added link 29, mass 0.24003132671428143; collision cylinder length=0.8673625771967088 radius=0.29679643923896615; visual cylinder length=0.8673625771967088 radius=0.29679643923896615
Joints:
- removed joint base_to_sub
- removed joint base_to_sub2
- added joint 11_to_0: type revolute, parent 0, child 11, origin xyz=0.10327429382701014 0.2744962115940697 0.9988360916566166 rpy=7.123823405232995 1.47491114932513 6.257798842348477, axis 1 0 0, limit lower=3.1415 upper=-3.1415 effort=1 velocity=1
- added joint 14_to_0: type revolute, parent 0, child 14, origin xyz=0.10327429382701014 0.2744962115940697 0.9988360916566166 rpy=10.685735107849492 1.47491114932513 6.257798842348477, axis 1 0 0, limit lower=3.1415 upper=-3.1415 effort=1 velocity=1
- added joint 17_to_0: type revolute, parent 0, child 17, origin xyz=0.10327429382701014 0.2744962115940697 0.9988360916566166 rpy=14.24764681046599 1.47491114932513 6.257798842348477, axis 1 0 0, limit lower=3.1415 upper=-3.1415 effort=1 velocity=1
- added joint 22_to_11: type revolute, parent 11, child 22, origin xyz=0.49595651231659 0.7346387449013257 0.24987987611381013 rpy=4.4244311910705205 5.525695045881102 2.6521069068000354, axis 0 0 1, limit lower=3.1415 upper=-3.1415 effort=1 velocity=1
- added joint 23_to_11: type revolute, parent 11, child 23, origin xyz=0.49595651231659 0.7346387449013257 0.24987987611381013 rpy=6.63664678660578 5.525695045881102 2.6521069068000354, axis 0 0 1, limit lower=3.1415 upper=-3.1415 effort=1 velocity=1
- added joint 25_to_14: type revolute, parent 14, child 25, origin xyz=0.49595651231659 0.7346387449013257 0.24987987611381013 rpy=4.4244311910705205 5.525695045881102 2.6521069068000354, axis 0 0 1, limit lower=3.1415 upper=-3.1415 effort=1 velocity=1
- added joint 26_to_14: type revolute, parent 14, child 26, origin xyz=0.49595651231659 0.7346387449013257 0.24987987611381013 rpy=6.63664678660578 5.525695045881102 2.6521069068000354, axis 0 0 1, limit lower=3.1415 upper=-3.1415 effort=1 velocity=1
- added joint 28_to_17: type revolute, parent 17, child 28, origin xyz=0.49595651231659 0.7346387449013257 0.24987987611381013 rpy=4.4244311910705205 5.525695045881102 2.6521069068000354, axis 0 0 1, limit lower=3.1415 upper=-3.1415 effort=1 velocity=1
- added joint 29_to_17: type revolute, parent 17, child 29, origin xyz=0.49595651231659 0.7346387449013257 0.24987987611381013 rpy=6.63664678660578 5.525695045881102 2.6521069068000354, axis 0 0 1, limit lower=3.1415 upper=-3.1415 effort=1 velocity=1
