Commit message: automated series of testing created for hyperparameters. data collection regarding fittest creatures for each generation in each hyperparameter adjusted simulation

File: temp0.urdf (robot description, URDF)
Before this commit: robot pepe, 4 links, 3 joints
Links:
- removed link 12
- removed link 13
- added link 22, mass 0.7201272939641289; collision cylinder length=0.4992144062714243 radius=0.6776198890848838; visual cylinder length=0.4992144062714243 radius=0.6776198890848838
- link 0: mass 1.0563237823933445 -> 0.5598146897605916; geometry collision cylinder length=1.620270057947925 radius=0.33162976685398904; visual cylinder length=1.620270057947925 radius=0.33162976685398904
- link 11: mass 0.14897223855170239 -> 0.12977987995971638; geometry collision cylinder length=0.9839968931008223 radius=0.20489524701403172; visual cylinder length=0.9839968931008223 radius=0.20489524701403172
Joints:
- removed joint 12_to_0
- removed joint 13_to_0
- added joint 22_to_0: type revolute, parent 0, child 22, origin xyz=0.9999 0.7238567635861478 0.5522377714191339 rpy=5.558661727454597 2.5399956445500633 4.67058598033998, axis 0 1 0, limit lower=3.1415 upper=-3.1415 effort=1 velocity=1
- joint 11_to_0: origin xyz=0.4395348609760371 0.5167789386225082 0.8235360944058471 rpy=12.277245561587007 5.66721228121419 3.2352878676311425 -> xyz=0.5433014881025203 0.10072810275251065 0.7749395988028834 rpy=7.300555879291387 4.803052681363918 0.9855001705750575

Commit message: 50 iterations box and cylinder, automated

File: temp0.urdf (robot description, URDF)
Before this commit: robot pepe, 3 links, 2 joints
Links:
- removed link 22
- added link 12, mass 6.281300540076709; collision box size=1.9998 1.9998 1.9998; visual box size=1.9998 1.9998 1.9998
- added link 13, mass 6.281300540076709; collision box size=1.9998 1.9998 1.9998; visual box size=1.9998 1.9998 1.9998
- link 0: mass 0.5598146897605916 -> 6.281300540076709; geometry collision box size=1.9998 1.9998 1.9998; visual box size=1.9998 1.9998 1.9998
- link 11: mass 0.12977987995971638 -> 6.281300540076709; geometry collision box size=1.9998 1.9998 1.9998; visual box size=1.9998 1.9998 1.9998
Joints:
- removed joint 22_to_0
- added joint 12_to_0: type revolute, parent 0, child 12, origin xyz=0.9999 0.9999 0.9999 rpy=18.847670965946605 6.282556988648868 6.282556988648868, axis 0 0 1, limit lower=3.1415 upper=-3.1415 effort=1 velocity=1
- added joint 13_to_0: type revolute, parent 0, child 13, origin xyz=0.9999 0.9999 0.9999 rpy=25.130227954595473 6.282556988648868 6.282556988648868, axis 0 0 1, limit lower=3.1415 upper=-3.1415 effort=1 velocity=1
- joint 11_to_0: origin xyz=0.5433014881025203 0.10072810275251065 0.7749395988028834 rpy=7.300555879291387 4.803052681363918 0.9855001705750575 -> xyz=0.9999 0.9999 0.9999 rpy=12.565113977297736 6.282556988648868 6.282556988648868

Commit message: analysis on data started and has informed on further experiments

File: temp0.urdf (robot description, URDF)
Before this commit: robot pepe, 4 links, 3 joints
Links:
- added link 24, mass 6.281300540076709; collision sphere radius=0.9999; visual sphere radius=0.9999
- added link 25, mass 6.281300540076709; collision sphere radius=0.9999; visual sphere radius=0.9999
- added link 26, mass 6.281300540076709; collision sphere radius=0.9999; visual sphere radius=0.9999
- link 0: mass 6.281300540076709 -> 1.4059517815846734; geometry collision sphere radius=0.5676302569906508; visual sphere radius=0.5676302569906508
- link 11: geometry collision sphere radius=0.9999; visual sphere radius=0.9999
- link 12: geometry collision sphere radius=0.9999; visual sphere radius=0.9999
- link 13: geometry collision sphere radius=0.9999; visual sphere radius=0.9999
Joints:
- added joint 24_to_0: type revolute, parent 0, child 24, origin xyz=0.6330046434101493 0.6834813684812228 0.9999 rpy=31.41278494324434 6.282556988648868 2.519441459209564, axis 0 0 1, limit lower=3.1415 upper=-3.1415 effort=1 velocity=1
- added joint 25_to_0: type revolute, parent 0, child 25, origin xyz=0.6330046434101493 0.6834813684812228 0.9999 rpy=37.69534193189321 6.282556988648868 2.519441459209564, axis 0 0 1, limit lower=3.1415 upper=-3.1415 effort=1 velocity=1
- added joint 26_to_0: type revolute, parent 0, child 26, origin xyz=0.6330046434101493 0.6834813684812228 0.9999 rpy=43.977898920542074 6.282556988648868 2.519441459209564, axis 0 0 1, limit lower=3.1415 upper=-3.1415 effort=1 velocity=1
- joint 11_to_0: origin xyz=0.9999 0.9999 0.9999 rpy=12.565113977297736 6.282556988648868 6.282556988648868 -> xyz=0.9999 0.9999 0.9999 rpy=12.565113977297736 4.2063083140344935 6.282556988648868
- joint 12_to_0: origin xyz=0.9999 0.9999 0.9999 rpy=18.847670965946605 6.282556988648868 6.282556988648868 -> xyz=0.9999 0.9999 0.9999 rpy=18.847670965946605 4.2063083140344935 6.282556988648868
- joint 13_to_0: origin xyz=0.9999 0.9999 0.9999 rpy=25.130227954595473 6.282556988648868 6.282556988648868 -> xyz=0.9999 0.9999 0.9999 rpy=25.130227954595473 4.2063083140344935 6.282556988648868

File: test.urdf (robot description, URDF)
Before this commit: robot pepe, 103 links, 102 joints
Links:
- removed link 1026
- removed link 1053
- removed link 1080
- removed link 1127
- removed link 1128
- removed link 1154
- removed link 1155
- removed link 1181
- removed link 1182
- removed link 1289
- removed link 1390
- removed link 1413
- removed link 1414
- removed link 1415
- removed link 1420
- removed link 1421
- removed link 1422
- removed link 1433
- removed link 1434
- removed link 1435
- removed link 1440
- removed link 1441
- removed link 1442
- removed link 1447
- removed link 1448
- removed link 1449
- removed link 146
- removed link 1460
- removed link 1461
- removed link 1462
- removed link 1467
- removed link 1468
- removed link 1469
- removed link 147
- removed link 1474
- removed link 1475
- removed link 1476
- removed link 148
- removed link 1510
- removed link 1511
- removed link 1516
- removed link 1517
- removed link 1518
- removed link 1523
- removed link 1524
- removed link 1525
- removed link 1536
- removed link 1537
- removed link 1538
- removed link 1543
- removed link 1544
- removed link 1545
- removed link 1550
- removed link 1551
- removed link 1552
- removed link 1563
- removed link 1564
- removed link 1565
- removed link 1570
- removed link 1571
- removed link 1572
- removed link 1577
- removed link 1578
- removed link 1579
- removed link 159
- removed link 1697
- removed link 1698
- removed link 1794
- removed link 1795
- removed link 1796
- removed link 18100
- removed link 18101
- removed link 1899
- removed link 1991
- removed link 1992
- removed link 1993
- removed link 22
- removed link 229
- removed link 256
- removed link 33
- removed link 330
- removed link 331
- removed link 34
- removed link 357
- removed link 358
- removed link 486
- removed link 583
- removed link 584
- removed link 585
- removed link 687
- removed link 7102
- removed link 812
- removed link 819
- removed link 832
- removed link 839
- removed link 846
- removed link 85
- removed link 859
- removed link 866
- removed link 873
- removed link 988
- added link 12, mass 0.000658348583703179; collision cylinder length=1.51448108483691 radius=0.011763081057244662; visual cylinder length=1.51448108483691 radius=0.011763081057244662
- added link 13, mass 0.000658348583703179; collision cylinder length=1.51448108483691 radius=0.011763081057244662; visual cylinder length=1.51448108483691 radius=0.011763081057244662
- added link 24, mass 0.943617257292961; collision cylinder length=0.32450945922425434 radius=0.9620758668207081; visual cylinder length=0.32450945922425434 radius=0.9620758668207081
- link 0: mass 1.1681372134988606 -> 0.0005210269576047729; geometry collision cylinder length=0.9609004824837803 radius=0.013137597584303218; visual cylinder length=0.9609004824837803 radius=0.013137597584303218
- link 11: mass 2.327346718066652 -> 0.000658348583703179; geometry collision cylinder length=1.51448108483691 radius=0.011763081057244662; visual cylinder length=1.51448108483691 radius=0.011763081057244662
Joints:
- removed joint 1026_to_22
- removed joint 1053_to_229
- removed joint 1080_to_256
- removed joint 1127_to_22
- removed joint 1128_to_22
- removed joint 1154_to_229
- removed joint 1155_to_229
- removed joint 1181_to_256
- removed joint 1182_to_256
- removed joint 1289_to_988
- removed joint 1390_to_1289
- removed joint 1413_to_812
- removed joint 1414_to_812
- removed joint 1415_to_812
- removed joint 1420_to_819
- removed joint 1421_to_819
- removed joint 1422_to_819
- removed joint 1433_to_832
- removed joint 1434_to_832
- removed joint 1435_to_832
- removed joint 1440_to_839
- removed joint 1441_to_839
- removed joint 1442_to_839
- removed joint 1447_to_846
- removed joint 1448_to_846
- removed joint 1449_to_846
- removed joint 1460_to_859
- removed joint 1461_to_859
- removed joint 1462_to_859
- removed joint 1467_to_866
- removed joint 1468_to_866
- removed joint 1469_to_866
- removed joint 146_to_85
- removed joint 1474_to_873
- removed joint 1475_to_873
- removed joint 1476_to_873
- removed joint 147_to_85
- removed joint 148_to_85
- removed joint 1510_to_85
- removed joint 1511_to_85
- removed joint 1516_to_812
- removed joint 1517_to_812
- removed joint 1518_to_812
- removed joint 1523_to_819
- removed joint 1524_to_819
- removed joint 1525_to_819
- removed joint 1536_to_832
- removed joint 1537_to_832
- removed joint 1538_to_832
- removed joint 1543_to_839
- removed joint 1544_to_839
- removed joint 1545_to_839
- removed joint 1550_to_846
- removed joint 1551_to_846
- removed joint 1552_to_846
- removed joint 1563_to_859
- removed joint 1564_to_859
- removed joint 1565_to_859
- removed joint 1570_to_866
- removed joint 1571_to_866
- removed joint 1572_to_866
- removed joint 1577_to_873
- removed joint 1578_to_873
- removed joint 1579_to_873
- removed joint 159_to_85
- removed joint 1697_to_486
- removed joint 1698_to_486
- removed joint 1794_to_1289
- removed joint 1795_to_1289
- removed joint 1796_to_1289
- removed joint 18100_to_486
- removed joint 18101_to_486
- removed joint 1899_to_486
- removed joint 1991_to_1390
- removed joint 1992_to_1390
- removed joint 1993_to_1390
- removed joint 229_to_11
- removed joint 22_to_11
- removed joint 256_to_11
- removed joint 330_to_229
- removed joint 331_to_229
- removed joint 33_to_22
- removed joint 34_to_22
- removed joint 357_to_256
- removed joint 358_to_256
- removed joint 486_to_0
- removed joint 583_to_11
- removed joint 584_to_11
- removed joint 585_to_11
- removed joint 687_to_486
- removed joint 7102_to_0
- removed joint 812_to_22
- removed joint 819_to_22
- removed joint 832_to_229
- removed joint 839_to_229
- removed joint 846_to_229
- removed joint 859_to_256
- removed joint 85_to_22
- removed joint 866_to_256
- removed joint 873_to_256
- removed joint 988_to_687
- added joint 12_to_0: type revolute, parent 0, child 12, origin xyz=0.6528362011378711 0.4607239150175825 0.5593860552195509 rpy=0.6367766989334194 5.730012498366459 5.085601574083224, axis 1 0 0, limit lower=3.1415 upper=-3.1415 effort=1 velocity=1
- added joint 13_to_0: type revolute, parent 0, child 13, origin xyz=0.6528362011378711 0.4607239150175825 0.5593860552195509 rpy=0.8490355985778925 5.730012498366459 5.085601574083224, axis 1 0 0, limit lower=3.1415 upper=-3.1415 effort=1 velocity=1
- added joint 24_to_0: type revolute, parent 0, child 24, origin xyz=0.12276982652981785 0.3020976403086859 0.8577477283935233 rpy=8.082642464734144 0.4726102174015297 4.418943105349465, axis 0 0 1, limit lower=3.1415 upper=-3.1415 effort=1 velocity=1
- joint 11_to_0: origin xyz=0.658163310852489 0.22265241266991875 0.09560250707341089 rpy=3.9265834959141923 4.683641603159373 1.3223151204610664 -> xyz=0.6528362011378711 0.4607239150175825 0.5593860552195509 rpy=0.42451779928894623 5.730012498366459 5.085601574083224

Commit message: report started

File: temp0.urdf (robot description, URDF)
Before this commit: robot pepe, 130 links, 129 joints
Links:
- removed link 144
- removed link 187
- removed link 2102
- removed link 2116
- removed link 216
- removed link 230
- removed link 245
- removed link 259
- removed link 273
- removed link 288
- removed link 3103
- removed link 3117
- removed link 317
- removed link 33
- removed link 331
- removed link 346
- removed link 360
- removed link 374
- removed link 389
- removed link 4104
- removed link 4108
- removed link 4112
- removed link 4118
- removed link 412
- removed link 4122
- removed link 4126
- removed link 418
- removed link 422
- removed link 426
- removed link 432
- removed link 436
- removed link 44
- removed link 440
- removed link 447
- removed link 451
- removed link 455
- removed link 461
- removed link 465
- removed link 469
- removed link 475
- removed link 479
- removed link 48
- removed link 483
- removed link 490
- removed link 494
- removed link 498
- removed link 510
- removed link 5100
- removed link 5101
- removed link 5105
- removed link 5106
- removed link 5107
- removed link 5109
- removed link 511
- removed link 5110
- removed link 5111
- removed link 5113
- removed link 5114
- removed link 5115
- removed link 5119
- removed link 5120
- removed link 5121
- removed link 5123
- removed link 5124
- removed link 5125
- removed link 5127
- removed link 5128
- removed link 5129
- removed link 513
- removed link 514
- removed link 515
- removed link 519
- removed link 520
- removed link 521
- removed link 523
- removed link 524
- removed link 525
- removed link 527
- removed link 528
- removed link 529
- removed link 533
- removed link 534
- removed link 535
- removed link 537
- removed link 538
- removed link 539
- removed link 541
- removed link 542
- removed link 543
- removed link 548
- removed link 549
- removed link 55
- removed link 550
- removed link 552
- removed link 553
- removed link 554
- removed link 556
- removed link 557
- removed link 558
- removed link 56
- removed link 562
- removed link 563
- removed link 564
- removed link 566
- removed link 567
- removed link 568
- removed link 57
- removed link 570
- removed link 571
- removed link 572
- removed link 576
- removed link 577
- removed link 578
- removed link 580
- removed link 581
- removed link 582
- removed link 584
- removed link 585
- removed link 586
- removed link 59
- removed link 591
- removed link 592
- removed link 593
- removed link 595
- removed link 596
- removed link 597
- removed link 599
- added link 13, mass 0.0973956192422835; collision box size=1.6793171824580089 1.6793171824580089 1.6793171824580089; visual box size=1.6793171824580089 1.6793171824580089 1.6793171824580089
- added link 15, mass 0.0973956192422835; collision box size=1.6793171824580089 1.6793171824580089 1.6793171824580089; visual box size=1.6793171824580089 1.6793171824580089 1.6793171824580089
- added link 24, mass 0.011234846404056805; collision cylinder length=0.007805902181151625 radius=0.6768572436038026; visual cylinder length=0.007805902181151625 radius=0.6768572436038026
- added link 26, mass 0.011234846404056805; collision cylinder length=0.007805902181151625 radius=0.6768572436038026; visual cylinder length=0.007805902181151625 radius=0.6768572436038026
- link 0: mass 2.433658513279265 -> 0.27104816631840367; geometry collision box size=1.4422837028967659 1.4422837028967659 1.4422837028967659; visual box size=1.4422837028967659 1.4422837028967659 1.4422837028967659
- link 11: mass 0.8862245479835859 -> 0.0973956192422835; geometry collision box size=1.6793171824580089 1.6793171824580089 1.6793171824580089; visual box size=1.6793171824580089 1.6793171824580089 1.6793171824580089
- link 22: mass 2.3615934314283016 -> 0.011234846404056805; geometry collision cylinder length=0.007805902181151625 radius=0.6768572436038026; visual cylinder length=0.007805902181151625 radius=0.6768572436038026
Joints:
- removed joint 144_to_0
- removed joint 187_to_0
- removed joint 2102_to_187
- removed joint 2116_to_187
- removed joint 216_to_11
- removed joint 230_to_11
- removed joint 245_to_144
- removed joint 259_to_144
- removed joint 273_to_144
- removed joint 288_to_187
- removed joint 3103_to_2102
- removed joint 3117_to_2116
- removed joint 317_to_216
- removed joint 331_to_230
- removed joint 33_to_22
- removed joint 346_to_245
- removed joint 360_to_259
- removed joint 374_to_273
- removed joint 389_to_288
- removed joint 4104_to_2102
- removed joint 4108_to_2102
- removed joint 4112_to_2102
- removed joint 4118_to_2116
- removed joint 4122_to_2116
- removed joint 4126_to_2116
- removed joint 412_to_22
- removed joint 418_to_216
- removed joint 422_to_216
- removed joint 426_to_216
- removed joint 432_to_230
- removed joint 436_to_230
- removed joint 440_to_230
- removed joint 447_to_245
- removed joint 44_to_22
- removed joint 451_to_245
- removed joint 455_to_245
- removed joint 461_to_259
- removed joint 465_to_259
- removed joint 469_to_259
- removed joint 475_to_273
- removed joint 479_to_273
- removed joint 483_to_273
- removed joint 48_to_22
- removed joint 490_to_288
- removed joint 494_to_288
- removed joint 498_to_288
- removed joint 5100_to_498
- removed joint 5101_to_498
- removed joint 5105_to_4104
- removed joint 5106_to_4104
- removed joint 5107_to_4104
- removed joint 5109_to_4108
- removed joint 510_to_48
- removed joint 5110_to_4108
- removed joint 5111_to_4108
- removed joint 5113_to_4112
- removed joint 5114_to_4112
- removed joint 5115_to_4112
- removed joint 5119_to_4118
- removed joint 511_to_48
- removed joint 5120_to_4118
- removed joint 5121_to_4118
- removed joint 5123_to_4122
- removed joint 5124_to_4122
- removed joint 5125_to_4122
- removed joint 5127_to_4126
- removed joint 5128_to_4126
- removed joint 5129_to_4126
- removed joint 513_to_412
- removed joint 514_to_412
- removed joint 515_to_412
- removed joint 519_to_418
- removed joint 520_to_418
- removed joint 521_to_418
- removed joint 523_to_422
- removed joint 524_to_422
- removed joint 525_to_422
- removed joint 527_to_426
- removed joint 528_to_426
- removed joint 529_to_426
- removed joint 533_to_432
- removed joint 534_to_432
- removed joint 535_to_432
- removed joint 537_to_436
- removed joint 538_to_436
- removed joint 539_to_436
- removed joint 541_to_440
- removed joint 542_to_440
- removed joint 543_to_440
- removed joint 548_to_447
- removed joint 549_to_447
- removed joint 550_to_447
- removed joint 552_to_451
- removed joint 553_to_451
- removed joint 554_to_451
- removed joint 556_to_455
- removed joint 557_to_455
- removed joint 558_to_455
- removed joint 55_to_44
- removed joint 562_to_461
- removed joint 563_to_461
- removed joint 564_to_461
- removed joint 566_to_465
- removed joint 567_to_465
- removed joint 568_to_465
- removed joint 56_to_44
- removed joint 570_to_469
- removed joint 571_to_469
- removed joint 572_to_469
- removed joint 576_to_475
- removed joint 577_to_475
- removed joint 578_to_475
- removed joint 57_to_44
- removed joint 580_to_479
- removed joint 581_to_479
- removed joint 582_to_479
- removed joint 584_to_483
- removed joint 585_to_483
- removed joint 586_to_483
- removed joint 591_to_490
- removed joint 592_to_490
- removed joint 593_to_490
- removed joint 595_to_494
- removed joint 596_to_494
- removed joint 597_to_494
- removed joint 599_to_498
- removed joint 59_to_48
- added joint 13_to_0: type revolute, parent 0, child 13, origin xyz=0.13373472983671186 0.29737354379756853 0.6621108903792577 rpy=15.471448276388085 3.815832006601965 6.257160855174368, axis 0 1 0, limit lower=3.1415 upper=-3.1415 effort=1 velocity=1
- added joint 15_to_0: type revolute, parent 0, child 15, origin xyz=0.13373472983671186 0.29737354379756853 0.6621108903792577 rpy=20.62859770185078 3.815832006601965 6.257160855174368, axis 0 1 0, limit lower=3.1415 upper=-3.1415 effort=1 velocity=1
- added joint 24_to_13: type revolute, parent 13, child 24, origin xyz=0.44640277226779224 0.35296108024940176 0.5997270566348657 rpy=5.67668857185224 4.826414115524076 5.02613044416073, axis 0 1 0, limit lower=3.1415 upper=-3.1415 effort=1 velocity=1
- added joint 26_to_15: type revolute, parent 15, child 26, origin xyz=0.44640277226779224 0.35296108024940176 0.5997270566348657 rpy=5.67668857185224 4.826414115524076 5.02613044416073, axis 0 1 0, limit lower=3.1415 upper=-3.1415 effort=1 velocity=1
- joint 11_to_0: origin xyz=0.005096555782734602 0.11978472283039487 0.28889542575000915 rpy=12.35483736540991 6.150867155797274 5.514166033265675 -> xyz=0.13373472983671186 0.29737354379756853 0.6621108903792577 rpy=10.31429885092539 3.815832006601965 6.257160855174368
- joint 22_to_11: origin xyz=0.34604144637492684 0.9486809796451484 0.6204757887286447 rpy=11.477647711201918 2.9386225977356184 3.6706140324167555 -> xyz=0.44640277226779224 0.35296108024940176 0.5997270566348657 rpy=5.67668857185224 4.826414115524076 5.02613044416073

File: test.urdf (robot description, URDF)
Before this commit: robot pepe, 5 links, 4 joints
Links:
- removed link 12
- removed link 13
- removed link 24
- added link 22, mass 1.4553346520393262; collision sphere radius=0.6566744377234808; visual sphere radius=0.6566744377234808
- added link 23, mass 1.4553346520393262; collision sphere radius=0.6566744377234808; visual sphere radius=0.6566744377234808
- link 0: mass 0.0005210269576047729 -> 0.3570276566550985; geometry collision sphere radius=0.25356733159367595; visual sphere radius=0.25356733159367595
- link 11: mass 0.000658348583703179 -> 0.8165082980717001; geometry collision sphere radius=0.7276920202001341; visual sphere radius=0.7276920202001341
Joints:
- removed joint 12_to_0
- removed joint 13_to_0
- removed joint 24_to_0
- added joint 22_to_11: type revolute, parent 11, child 22, origin xyz=0.6782605252597379 0.6844388837015243 0.34435280458399986 rpy=12.565113977297736 6.282556988648868 6.282556988648868, axis 0 1 0, limit lower=3.1415 upper=-3.1415 effort=1 velocity=1
- added joint 23_to_11: type revolute, parent 11, child 23, origin xyz=0.6782605252597379 0.6844388837015243 0.34435280458399986 rpy=18.847670965946605 6.282556988648868 6.282556988648868, axis 0 1 0, limit lower=3.1415 upper=-3.1415 effort=1 velocity=1
- joint 11_to_0: origin xyz=0.6528362011378711 0.4607239150175825 0.5593860552195509 rpy=0.42451779928894623 5.730012498366459 5.085601574083224 -> xyz=0.9833797638016106 0.9180415406468643 0.984771766238487 rpy=9.230303782013191 4.51120824161145 4.575930900816994
