Commit message: further focussed exploration of hyperparameter effects

File: temp0.urdf (robot description, URDF)
Before this commit: robot pepe, 7 links, 6 joints
Links:
- removed link 13
- removed link 15
- removed link 22
- removed link 24
- removed link 26
- added link 12, mass 6.281300540076709; collision cylinder length=1.9998 radius=0.9999; visual cylinder length=1.9998 radius=0.9999
- link 0: mass 0.27104816631840367 -> 0.002428490064569883; geometry collision box size=1.6322319111498327 1.6322319111498327 1.6322319111498327; visual box size=1.6322319111498327 1.6322319111498327 1.6322319111498327
- link 11: mass 0.0973956192422835 -> 6.281300540076709; geometry collision cylinder length=1.9998 radius=0.9999; visual cylinder length=1.9998 radius=0.9999
Joints:
- removed joint 13_to_0
- removed joint 15_to_0
- removed joint 22_to_11
- removed joint 24_to_13
- removed joint 26_to_15
- added joint 12_to_0: type revolute, parent 0, child 12, origin xyz=0.06904317670072035 0.9999 0.8026076203724806 rpy=18.847670965946605 3.600420847499156 2.982406471367985, axis 0 0 1, limit lower=3.1415 upper=-3.1415 effort=1 velocity=1
- joint 11_to_0: axis 0 1 0 -> 0 0 1; origin xyz=0.13373472983671186 0.29737354379756853 0.6621108903792577 rpy=10.31429885092539 3.815832006601965 6.257160855174368 -> xyz=0.06904317670072035 0.9999 0.8026076203724806 rpy=12.565113977297736 3.600420847499156 2.982406471367985

File: test.urdf (robot description, URDF)
Before this commit: robot pepe, 4 links, 3 joints
Links:
- removed link 23
- link 0: mass 0.3570276566550985 -> 0.016432958793730097; geometry collision sphere radius=0.6429822244510458; visual sphere radius=0.6429822244510458
- link 11: mass 0.8165082980717001 -> 0.8753884536007785; geometry collision sphere radius=0.45409667178427515; visual sphere radius=0.45409667178427515
- link 22: mass 1.4553346520393262 -> 5.706928602310837; geometry collision box size=1.8169351627237753 1.8169351627237753 1.8169351627237753; visual box size=1.8169351627237753 1.8169351627237753 1.8169351627237753
Joints:
- removed joint 23_to_11
- joint 11_to_0: origin xyz=0.9833797638016106 0.9180415406468643 0.984771766238487 rpy=9.230303782013191 4.51120824161145 4.575930900816994 -> xyz=0.3654569990874831 0.2625542508417571 0.7669329391729968 rpy=5.816286777877302 1.2449199875318697 4.153128970209793
- joint 22_to_11: axis 0 1 0 -> 0 0 1; origin xyz=0.6782605252597379 0.6844388837015243 0.34435280458399986 rpy=12.565113977297736 6.282556988648868 6.282556988648868 -> xyz=0.3621430780854923 0.8833197334664157 0.7715773064837551 rpy=1.8103414222245964 5.276144194749023 4.678265846527187
